File: blinkyProject.sch (KiCad schematic (older format))
At the start: 12 parts

Commit message: Annotates schematic
Parts:
- gave numbers to parts that had none: 12
Changed lines of the file:
@@
 $EndDescr
 $Comp
-L MCU_ST_STM32F0-custom:stm32f030 U??
-U 1 1 60FC94A6
-P 5100 4100
-F 0 "U??" H 5100 4700 50  0000 C CNN
-F 1 "stm32f030" H 5100 3500 50  0000 C CNN
-F 2 "" H 5000 3150 50  0001 C CNN
-F 3 "" H 5000 3150 50  0001 C CNN
-	1    5100 4100
-	1    0    0    -1
-$EndComp
-$Comp
-L Device:C_Small C?
+L Device:C_Small C2
 U 1 1 60FD214B
 P 3750 3600
-F 0 "C?" H 3842 3646 50  0000 L CNN
+F 0 "C2" H 3842 3646 50  0000 L CNN
 F 1 "0.1uF" H 3842 3555 50  0000 L CNN
 F 2 "" H 3750 3600 50  0001 C CNN
@@
 $EndComp
 $Comp
-L Device:C_Small C?
+L Device:C_Small C3
 U 1 1 60FD2C0F
 P 3950 4150
-F 0 "C?" H 4042 4196 50  0000 L CNN
+F 0 "C3" H 4042 4196 50  0000 L CNN
 F 1 "1uF" H 4042 4105 50  0000 L CNN
 F 2 "" H 3950 4150 50  0001 C CNN
@@
 $EndComp
 $Comp
-L Device:C_Small C?
+L Device:C_Small C4
 U 1 1 60FD2F1F
 P 6650 4200
-F 0 "C?" H 6742 4246 50  0000 L CNN
+F 0 "C4" H 6742 4246 50  0000 L CNN
 F 1 "100nF" H 6742 4155 50  0000 L CNN
 F 2 "" H 6650 4200 50  0001 C CNN
@@
 $EndComp
 $Comp
-L Device:C_Small C?
+L Device:C_Small C1
 U 1 1 60FD310A
 P 3500 4150
-F 0 "C?" H 3592 4196 50  0000 L CNN
+F 0 "C1" H 3592 4196 50  0000 L CNN
 F 1 "10nF" H 3592 4105 50  0000 L CNN
 F 2 "" H 3500 4150 50  0001 C CNN
@@
 $EndComp
 $Comp
-L Device:C_Small C?
+L Device:C_Small C5
 U 1 1 60FD40EB
 P 7100 4200
-F 0 "C?" H 7192 4246 50  0000 L CNN
+F 0 "C5" H 7192 4246 50  0000 L CNN
 F 1 "4.7uF" H 7192 4155 50  0000 L CNN
 F 2 "" H 7100 4200 50  0001 C CNN
@@
 $EndComp
 $Comp
-L Device:R R?
+L Device:R R1
 U 1 1 60FD4ACB
 P 7050 4950
-F 0 "R?" V 6843 4950 50  0000 C CNN
+F 0 "R1" V 6843 4950 50  0000 C CNN
 F 1 "39" V 7050 4950 50  0000 C CNN
 F 2 "" V 6980 4950 50  0001 C CNN
@@
 $EndComp
 $Comp
-L Device:LED D?
+L Device:LED D1
 U 1 1 60FD9142
 P 6600 4950
-F 0 "D?" H 6593 5167 50  0000 C CNN
+F 0 "D1" H 6593 5167 50  0000 C CNN
 F 1 "LED" H 6593 5076 50  0000 C CNN
 F 2 "" H 6600 4950 50  0001 C CNN
@@
 $EndComp
 $Comp
-L Device:R_Pack04 RN?
+L Device:R_Pack04 RN1
 U 1 1 60FD9B9C
 P 6300 3600
-F 0 "RN?" H 6488 3646 50  0000 L CNN
+F 0 "RN1" H 6488 3646 50  0000 L CNN
 F 1 "4.7k" H 6488 3555 50  0000 L CNN
 F 2 "" V 6575 3600 50  0001 C CNN
@@
 $EndComp
 $Comp
-L Regulator_Linear:LD1117S33TR_SOT223 U?
+L Regulator_Linear:LD1117S33TR_SOT223 U1
 U 1 1 60FDA95F
 P 6050 2250
-F 0 "U?" H 6050 2492 50  0000 C CNN
+F 0 "U1" H 6050 2492 50  0000 C CNN
 F 1 "LD1117S33TR_SOT223" H 6050 2401 50  0000 C CNN
 F 2 "Package_TO_SOT_SMD:SOT-223-3_TabPin2" H 6050 2450 50  0001 C CNN
@@
 $EndComp
 $Comp
-L Connector:USB_B_Micro J?
+L Connector:USB_B_Micro J1
 U 1 1 60FDB8CF
 P 7000 2450
-F 0 "J?" H 6770 2439 50  0000 R CNN
+F 0 "J1" H 6770 2439 50  0000 R CNN
 F 1 "USB_B_Micro" H 6770 2348 50  0000 R CNN
 F 2 "" H 7150 2400 50  0001 C CNN
@@
 $EndComp
 $Comp
-L Connector_Generic:Conn_02x10_Odd_Even J?
+L Connector_Generic:Conn_02x10_Odd_Even J2
 U 1 1 60FDDC5B
 P 8150 4050
-F 0 "J?" H 8200 4667 50  0000 C CNN
+F 0 "J2" H 8200 4667 50  0000 C CNN
 F 1 "Conn_02x10_Odd_Even" H 8200 4576 50  0000 C CNN
 F 2 "" H 8150 4050 50  0001 C CNN
@@
 $EndComp
 $Comp
-L power:+3.3V #PWR?
+L power:+3.3V #PWR01
 U 1 1 60FE2CCD
 P 3500 4000
-F 0 "#PWR?" H 3500 3850 50  0001 C CNN
+F 0 "#PWR01" H 3500 3850 50  0001 C CNN
 F 1 "+3.3V" H 3515 4173 50  0000 C CNN
 F 2 "" H 3500 4000 50  0001 C CNN
@@
 $EndComp
 $Comp
-L power:GND #PWR?
+L power:GND #PWR03
 U 1 1 60FE38EF
 P 3750 3800
-F 0 "#PWR?" H 3750 3550 50  0001 C CNN
+F 0 "#PWR03" H 3750 3550 50  0001 C CNN
 F 1 "GND" H 3755 3627 50  0000 C CNN
 F 2 "" H 3750 3800 50  0001 C CNN
@@
 $EndComp
 $Comp
-L power:GND #PWR?
+L power:GND #PWR05
 U 1 1 60FE5420
 P 4250 3700
-F 0 "#PWR?" H 4250 3450 50  0001 C CNN
+F 0 "#PWR05" H 4250 3450 50  0001 C CNN
 F 1 "GND" H 4255 3527 50  0000 C CNN
 F 2 "" H 4250 3700 50  0001 C CNN
@@
 Connection ~ 3500 4050
 $Comp
-L power:GND #PWR?
+L power:GND #PWR02
 U 1 1 60FEE816
 P 3500 4350
-F 0 "#PWR?" H 3500 4100 50  0001 C CNN
+F 0 "#PWR02" H 3500 4100 50  0001 C CNN
 F 1 "GND" H 3505 4177 50  0000 C CNN
 F 2 "" H 3500 4350 50  0001 C CNN
@@
 $EndComp
 $Comp
-L power:GND #PWR?
+L power:GND #PWR04
 U 1 1 60FEEB7A
 P 3950 4350
-F 0 "#PWR?" H 3950 4100 50  0001 C CNN
+F 0 "#PWR04" H 3950 4100 50  0001 C CNN
 F 1 "GND" H 3955 4177 50  0000 C CNN
 F 2 "" H 3950 4350 50  0001 C CNN
@@
 	3750 3500 4050 3500
 $Comp
-L power:+3.3V #PWR?
+L power:+3.3V #PWR014
 U 1 1 60FF4805
 P 7350 4850
-F 0 "#PWR?" H 7350 4700 50  0001 C CNN
+F 0 "#PWR014" H 7350 4700 50  0001 C CNN
 F 1 "+3.3V" H 7365 5023 50  0000 C CNN
 F 2 "" H 7350 4850 50  0001 C CNN
@@
 	6300 4950 6450 4950
 $Comp
-L power:GND #PWR?
+L power:GND #PWR09
 U 1 1 60FF81D8
 P 6400 4250
-F 0 "#PWR?" H 6400 4000 50  0001 C CNN
+F 0 "#PWR09" H 6400 4000 50  0001 C CNN
 F 1 "GND" H 6405 4077 50  0000 C CNN
 F 2 "" H 6400 4250 50  0001 C CNN
@@
 	6650 4050 7100 4050
 $Comp
-L power:+3.3V #PWR?
+L power:+3.3V #PWR012
 U 1 1 60FFB0D9
 P 7100 4000
-F 0 "#PWR?" H 7100 3850 50  0001 C CNN
+F 0 "#PWR012" H 7100 3850 50  0001 C CNN
 F 1 "+3.3V" H 7115 4173 50  0000 C CNN
 F 2 "" H 7100 4000 50  0001 C CNN
@@
 Connection ~ 7100 4050
 $Comp
-L power:GND #PWR?
+L power:GND #PWR010
 U 1 1 60FFBC5F
 P 6650 4400
-F 0 "#PWR?" H 6650 4150 50  0001 C CNN
+F 0 "#PWR010" H 6650 4150 50  0001 C CNN
 F 1 "GND" H 6655 4227 50  0000 C CNN
 F 2 "" H 6650 4400 50  0001 C CNN
@@
 	6650 4400 6650 4300
 $Comp
-L power:GND #PWR?
+L power:GND #PWR013
 U 1 1 60FFC640
 P 7100 4400
-F 0 "#PWR?" H 7100 4150 50  0001 C CNN
+F 0 "#PWR013" H 7100 4150 50  0001 C CNN
 F 1 "GND" H 7105 4227 50  0000 C CNN
 F 2 "" H 7100 4400 50  0001 C CNN
@@
 	6200 3850 6550 3850
 $Comp
-L power:+3.3V #PWR?
+L power:+3.3V #PWR08
 U 1 1 60FFFA9C
 P 6100 3300
-F 0 "#PWR?" H 6100 3150 50  0001 C CNN
+F 0 "#PWR08" H 6100 3150 50  0001 C CNN
 F 1 "+3.3V" H 6115 3473 50  0000 C CNN
 F 2 "" H 6100 3300 50  0001 C CNN
@@
 	6350 2250 6700 2250
 $Comp
-L power:+3.3V #PWR?
+L power:+3.3V #PWR06
 U 1 1 61002C6E
 P 5550 2200
-F 0 "#PWR?" H 5550 2050 50  0001 C CNN
+F 0 "#PWR06" H 5550 2050 50  0001 C CNN
 F 1 "+3.3V" H 5565 2373 50  0000 C CNN
 F 2 "" H 5550 2200 50  0001 C CNN
@@
 	5550 2250 5550 2200
 $Comp
-L power:GND #PWR?
+L power:GND #PWR07
 U 1 1 61003A7A
 P 6050 2650
-F 0 "#PWR?" H 6050 2400 50  0001 C CNN
+F 0 "#PWR07" H 6050 2400 50  0001 C CNN
 F 1 "GND" H 6055 2477 50  0000 C CNN
 F 2 "" H 6050 2650 50  0001 C CNN
@@
 	6050 2650 6050 2550
 $Comp
-L power:GND #PWR?
+L power:GND #PWR011
 U 1 1 61004D25
 P 7000 2950
-F 0 "#PWR?" H 7000 2700 50  0001 C CNN
+F 0 "#PWR011" H 7000 2700 50  0001 C CNN
 F 1 "GND" H 7005 2777 50  0000 C CNN
 F 2 "" H 7000 2950 50  0001 C CNN
@@
 Connection ~ 7000 2850
 $Comp
-L power:+3.3V #PWR?
+L power:+3.3V #PWR015
 U 1 1 6100B191
 P 7450 3600
-F 0 "#PWR?" H 7450 3450 50  0001 C CNN
+F 0 "#PWR015" H 7450 3450 50  0001 C CNN
 F 1 "+3.3V" H 7465 3773 50  0000 C CNN
 F 2 "" H 7450 3600 50  0001 C CNN
@@
 	7950 4150 7950 4050
 $Comp
-L power:GND #PWR?
+L power:GND #PWR016
 U 1 1 6100D74A
 P 7800 3750
-F 0 "#PWR?" H 7800 3500 50  0001 C CNN
+F 0 "#PWR016" H 7800 3500 50  0001 C CNN
 F 1 "GND" V 7805 3622 50  0000 R CNN
 F 2 "" H 7800 3750 50  0001 C CNN
@@
 ADC_IN1
 $Comp
-L power:GND #PWR?
+L power:GND #PWR017
 U 1 1 61012528
 P 7800 4550
-F 0 "#PWR?" H 7800 4300 50  0001 C CNN
+F 0 "#PWR017" H 7800 4300 50  0001 C CNN
 F 1 "GND" V 7805 4422 50  0000 R CNN
 F 2 "" H 7800 4550 50  0001 C CNN
@@
 NoConn ~ 6700 2550
 NoConn ~ 6700 2650
+$Comp
+L MCU_ST_STM32F0-custom:stm32f030 U1
+U 1 1 60FC94A6
+P 5100 4100
+F 0 "U1" H 5100 4700 50  0000 C CNN
+F 1 "stm32f030" H 5100 3500 50  0000 C CNN
+F 2 "" H 5000 3150 50  0001 C CNN
+F 3 "" H 5000 3150 50  0001 C CNN
+	1    5100 4100
+	1    0    0    -1
+$EndComp
 $EndSCHEMATC

Commit message: Generates Netlist
Parts:
- renumbered U1 to U2
Changed lines of the file:
@@
 $EndComp
 $Comp
-L Regulator_Linear:LD1117S33TR_SOT223 U1
+L Regulator_Linear:LD1117S33TR_SOT223 U2
 U 1 1 60FDA95F
 P 6050 2250
-F 0 "U1" H 6050 2492 50  0000 C CNN
+F 0 "U2" H 6050 2492 50  0000 C CNN
 F 1 "LD1117S33TR_SOT223" H 6050 2401 50  0000 C CNN
 F 2 "Package_TO_SOT_SMD:SOT-223-3_TabPin2" H 6050 2450 50  0001 C CNN

Commit message: Assigns footprints to schematic symbol
Parts:
- C1, C2, C3, C4, C5: footprint (none) -> Capacitor_SMD:C_0805_2012Metric_Pad1.18x1.45mm_HandSolder
- D1: footprint (none) -> LED_SMD:LED_0805_2012Metric_Pad1.15x1.40mm_HandSolder
- J1: footprint (none) -> Connector_USB:USB_Micro-B_Molex-105017-0001
- J2: footprint (none) -> Connector_PinHeader_2.54mm:PinHeader_2x10_P2.54mm_Vertical
- R1: footprint (none) -> Resistor_SMD:R_0805_2012Metric_Pad1.20x1.40mm_HandSolder
- RN1: footprint (none) -> Resistor_SMD:R_Array_Convex_4x0603
- U1: footprint (none) -> Package_SO:TSSOP-20_4.4x6.5mm_P0.65mm
Changed lines of the file:
@@
 F 0 "C2" H 3842 3646 50  0000 L CNN
 F 1 "0.1uF" H 3842 3555 50  0000 L CNN
-F 2 "" H 3750 3600 50  0001 C CNN
+F 2 "Capacitor_SMD:C_0805_2012Metric_Pad1.18x1.45mm_HandSolder" H 3750 3600 50  0001 C CNN
 F 3 "~" H 3750 3600 50  0001 C CNN
 	1    3750 3600
@@
 F 0 "C3" H 4042 4196 50  0000 L CNN
 F 1 "1uF" H 4042 4105 50  0000 L CNN
-F 2 "" H 3950 4150 50  0001 C CNN
+F 2 "Capacitor_SMD:C_0805_2012Metric_Pad1.18x1.45mm_HandSolder" H 3950 4150 50  0001 C CNN
 F 3 "~" H 3950 4150 50  0001 C CNN
 	1    3950 4150
@@
 F 0 "C4" H 6742 4246 50  0000 L CNN
 F 1 "100nF" H 6742 4155 50  0000 L CNN
-F 2 "" H 6650 4200 50  0001 C CNN
+F 2 "Capacitor_SMD:C_0805_2012Metric_Pad1.18x1.45mm_HandSolder" H 6650 4200 50  0001 C CNN
 F 3 "~" H 6650 4200 50  0001 C CNN
 	1    6650 4200
@@
 F 0 "C1" H 3592 4196 50  0000 L CNN
 F 1 "10nF" H 3592 4105 50  0000 L CNN
-F 2 "" H 3500 4150 50  0001 C CNN
+F 2 "Capacitor_SMD:C_0805_2012Metric_Pad1.18x1.45mm_HandSolder" H 3500 4150 50  0001 C CNN
 F 3 "~" H 3500 4150 50  0001 C CNN
 	1    3500 4150
@@
 F 0 "C5" H 7192 4246 50  0000 L CNN
 F 1 "4.7uF" H 7192 4155 50  0000 L CNN
-F 2 "" H 7100 4200 50  0001 C CNN
+F 2 "Capacitor_SMD:C_0805_2012Metric_Pad1.18x1.45mm_HandSolder" H 7100 4200 50  0001 C CNN
 F 3 "~" H 7100 4200 50  0001 C CNN
 	1    7100 4200
@@
 F 0 "R1" V 6843 4950 50  0000 C CNN
 F 1 "39" V 7050 4950 50  0000 C CNN
-F 2 "" V 6980 4950 50  0001 C CNN
+F 2 "Resistor_SMD:R_0805_2012Metric_Pad1.20x1.40mm_HandSolder" V 6980 4950 50  0001 C CNN
 F 3 "~" H 7050 4950 50  0001 C CNN
 	1    7050 4950
@@
 F 0 "D1" H 6593 5167 50  0000 C CNN
 F 1 "LED" H 6593 5076 50  0000 C CNN
-F 2 "" H 6600 4950 50  0001 C CNN
+F 2 "LED_SMD:LED_0805_2012Metric_Pad1.15x1.40mm_HandSolder" H 6600 4950 50  0001 C CNN
 F 3 "~" H 6600 4950 50  0001 C CNN
 	1    6600 4950
@@
 F 0 "RN1" H 6488 3646 50  0000 L CNN
 F 1 "4.7k" H 6488 3555 50  0000 L CNN
-F 2 "" V 6575 3600 50  0001 C CNN
+F 2 "Resistor_SMD:R_Array_Convex_4x0603" V 6575 3600 50  0001 C CNN
 F 3 "~" H 6300 3600 50  0001 C CNN
 	1    6300 3600
@@
 F 0 "J1" H 6770 2439 50  0000 R CNN
 F 1 "USB_B_Micro" H 6770 2348 50  0000 R CNN
-F 2 "" H 7150 2400 50  0001 C CNN
+F 2 "Connector_USB:USB_Micro-B_Molex-105017-0001" H 7150 2400 50  0001 C CNN
 F 3 "~" H 7150 2400 50  0001 C CNN
 	1    7000 2450
@@
 F 0 "J2" H 8200 4667 50  0000 C CNN
 F 1 "Conn_02x10_Odd_Even" H 8200 4576 50  0000 C CNN
-F 2 "" H 8150 4050 50  0001 C CNN
+F 2 "Connector_PinHeader_2.54mm:PinHeader_2x10_P2.54mm_Vertical" H 8150 4050 50  0001 C CNN
 F 3 "~" H 8150 4050 50  0001 C CNN
 	1    8150 4050
@@
 F 0 "U1" H 5100 4700 50  0000 C CNN
 F 1 "stm32f030" H 5100 3500 50  0000 C CNN
-F 2 "" H 5000 3150 50  0001 C CNN
+F 2 "Package_SO:TSSOP-20_4.4x6.5mm_P0.65mm" H 5000 3150 50  0001 C CNN
 F 3 "" H 5000 3150 50  0001 C CNN
 	1    5100 4100

Commit message: Adds capacitor C6 and C7
Parts:
- added C6, C7: 10uF, Capacitor_SMD:C_0805_2012Metric_Pad1.18x1.45mm_HandSolder, symbol Device:C_Small
Connections:
- net +3V3: now also C6.1
- net GND: now also C6.2, C7.2
- net +5V: now reaches J1.1 (VBUS), U2.3 (VI)
- net +5V: now also C7.1
Other:
- moved on the sheet: J1
Changed lines of the file:
@@
 L Connector:USB_B_Micro J1
 U 1 1 60FDB8CF
-P 7000 2450
-F 0 "J1" H 6770 2439 50  0000 R CNN
-F 1 "USB_B_Micro" H 6770 2348 50  0000 R CNN
-F 2 "Connector_USB:USB_Micro-B_Molex-105017-0001" H 7150 2400 50  0001 C CNN
-F 3 "~" H 7150 2400 50  0001 C CNN
-	1    7000 2450
+P 7100 2450
+F 0 "J1" H 6870 2439 50  0000 R CNN
+F 1 "USB_B_Micro" H 6870 2348 50  0000 R CNN
+F 2 "Connector_USB:USB_Micro-B_Molex-105017-0001" H 7250 2400 50  0001 C CNN
+F 3 "~" H 7250 2400 50  0001 C CNN
+	1    7100 2450
 	-1   0    0    -1
 $EndComp
@@
 Connection ~ 6100 3400
 Wire Wire Line
-	6350 2250 6700 2250
+	6350 2250 6450 2250
 $Comp
 L power:+3.3V #PWR06
@@
 $EndComp
 Wire Wire Line
-	5750 2250 5550 2250
+	5750 2250 5650 2250
 Wire Wire Line
 	5550 2250 5550 2200
@@
 L power:GND #PWR011
 U 1 1 61004D25
-P 7000 2950
-F 0 "#PWR011" H 7000 2700 50  0001 C CNN
-F 1 "GND" H 7005 2777 50  0000 C CNN
-F 2 "" H 7000 2950 50  0001 C CNN
-F 3 "" H 7000 2950 50  0001 C CNN
-	1    7000 2950
-	1    0    0    -1
-$EndComp
-Wire Wire Line
-	7000 2950 7000 2850
+P 7100 2950
+F 0 "#PWR011" H 7100 2700 50  0001 C CNN
+F 1 "GND" H 7105 2777 50  0000 C CNN
+F 2 "" H 7100 2950 50  0001 C CNN
+F 3 "" H 7100 2950 50  0001 C CNN
+	1    7100 2950
+	1    0    0    -1
+$EndComp
+Wire Wire Line
+	7100 2950 7100 2850
 Wire Wire Line
 	6100 3300 6100 3400
 Wire Wire Line
-	7000 2850 7100 2850
-Connection ~ 7000 2850
+	7100 2850 7200 2850
+Connection ~ 7100 2850
 $Comp
 L power:+3.3V #PWR015
@@
 NoConn ~ 6300 3400
 NoConn ~ 6400 3400
-NoConn ~ 6700 2450
-NoConn ~ 6700 2550
-NoConn ~ 6700 2650
+NoConn ~ 6800 2450
+NoConn ~ 6800 2550
+NoConn ~ 6800 2650
 $Comp
 L MCU_ST_STM32F0-custom:stm32f030 U1
@@
 	1    0    0    -1
 $EndComp
+$Comp
+L Device:C_Small C7
+U 1 1 6104012D
+P 6450 2500
+F 0 "C7" H 6542 2546 50  0000 L CNN
+F 1 "10uF" H 6542 2455 50  0000 L CNN
+F 2 "Capacitor_SMD:C_0805_2012Metric_Pad1.18x1.45mm_HandSolder" H 6450 2500 50  0001 C CNN
+F 3 "~" H 6450 2500 50  0001 C CNN
+	1    6450 2500
+	1    0    0    -1
+$EndComp
+$Comp
+L Device:C_Small C6
+U 1 1 61040C43
+P 5650 2500
+F 0 "C6" H 5742 2546 50  0000 L CNN
+F 1 "10uF" H 5742 2455 50  0000 L CNN
+F 2 "Capacitor_SMD:C_0805_2012Metric_Pad1.18x1.45mm_HandSolder" H 5650 2500 50  0001 C CNN
+F 3 "~" H 5650 2500 50  0001 C CNN
+	1    5650 2500
+	1    0    0    -1
+$EndComp
+$Comp
+L power:+5V #PWR020
+U 1 1 6104161C
+P 6600 2150
+F 0 "#PWR020" H 6600 2000 50  0001 C CNN
+F 1 "+5V" H 6615 2323 50  0000 C CNN
+F 2 "" H 6600 2150 50  0001 C CNN
+F 3 "" H 6600 2150 50  0001 C CNN
+	1    6600 2150
+	1    0    0    -1
+$EndComp
+Wire Wire Line
+	6600 2150 6600 2250
+Connection ~ 6600 2250
+Wire Wire Line
+	6450 2400 6450 2250
+Connection ~ 6450 2250
+Wire Wire Line
+	6450 2250 6600 2250
+Wire Wire Line
+	5650 2400 5650 2250
+Connection ~ 5650 2250
+Wire Wire Line
+	5650 2250 5550 2250
+$Comp
+L power:GND #PWR018
+U 1 1 610449B6
+P 5650 2700
+F 0 "#PWR018" H 5650 2450 50  0001 C CNN
+F 1 "GND" H 5655 2527 50  0000 C CNN
+F 2 "" H 5650 2700 50  0001 C CNN
+F 3 "" H 5650 2700 50  0001 C CNN
+	1    5650 2700
+	1    0    0    -1
+$EndComp
+$Comp
+L power:GND #PWR019
+U 1 1 61044D9B
+P 6450 2700
+F 0 "#PWR019" H 6450 2450 50  0001 C CNN
+F 1 "GND" H 6455 2527 50  0000 C CNN
+F 2 "" H 6450 2700 50  0001 C CNN
+F 3 "" H 6450 2700 50  0001 C CNN
+	1    6450 2700
+	1    0    0    -1
+$EndComp
+Wire Wire Line
+	6450 2700 6450 2600
+Wire Wire Line
+	5650 2700 5650 2600
+Wire Wire Line
+	6600 2250 6800 2250
 $EndSCHEMATC
