File: blinkyProject.sch (KiCad schematic (older format))
At the start: 14 parts, among them J1 USB_B_Micro, J2 Conn_02x10_Odd_Even, U1 stm32f030, U2 LD1117S33TR_SOT223

Commit message: Completes routing
Connections:
- net I2C1_SCL: now also J2.12 (Pin_12), RN1.2 (R2.1); no longer J2.11 (Pin_11), RN1.1 (R1.1)
- net I2C1_SDA: now also J2.11 (Pin_11), RN1.1 (R1.1); no longer J2.12 (Pin_12), RN1.2 (R2.1)
- net SPI1_MISO: now also J2.6 (Pin_6); no longer J2.7 (Pin_7)
- net SPI1_MOSI: now also J2.5 (Pin_5); no longer J2.8 (Pin_8)
- net SPI1_NSS: now also J2.8 (Pin_8); no longer J2.5 (Pin_5)
- net SPI1_SCK: now also J2.7 (Pin_7); no longer J2.6 (Pin_6)
- net SWCLK: now also J2.13 (Pin_13); no longer J2.14 (Pin_14)
- net SWDIO: now also J2.14 (Pin_14); no longer J2.13 (Pin_13)
- net USART1_RX: now also J2.18 (Pin_18); no longer J2.17 (Pin_17)
- net USART1_TX: now also J2.17 (Pin_17); no longer J2.18 (Pin_18)
Changed lines of the file:
@@
 Wire Wire Line
 	7100 4400 7100 4300
-Wire Wire Line
-	5600 3850 6200 3850
-Wire Wire Line
-	5600 3950 6100 3950
-Wire Wire Line
-	6100 3800 6100 3950
-Connection ~ 6100 3950
-Wire Wire Line
-	6100 3950 6550 3950
-Wire Wire Line
-	6200 3800 6200 3850
-Connection ~ 6200 3850
-Wire Wire Line
-	6200 3850 6550 3850
 $Comp
 L power:+3.3V #PWR08
@@
 	0    -1   -1   0
 $EndComp
+Text GLabel 8150 4250 0    50   Input ~ 0
+SWCLK
 Text GLabel 8650 4250 2    50   Input ~ 0
-SWCLK
-Text GLabel 8150 4250 0    50   Input ~ 0
 SWDIO
+Text GLabel 8150 4150 0    50   Input ~ 0
+I2C1_SDA
 Text GLabel 8650 4150 2    50   Input ~ 0
-I2C1_SDA
-Text GLabel 8150 4150 0    50   Input ~ 0
 I2C1_SCL
+Text GLabel 8650 3950 2    50   Input ~ 0
+SPI1_NSS
+Text GLabel 8150 3950 0    50   Input ~ 0
+SPI1_SCK
+Text GLabel 8650 3850 2    50   Input ~ 0
+SPI1_MISO
 Text GLabel 8150 3850 0    50   Input ~ 0
-SPI1_NSS
-Text GLabel 8650 3850 2    50   Input ~ 0
-SPI1_SCK
-Text GLabel 8150 3950 0    50   Input ~ 0
-SPI1_MISO
-Text GLabel 8650 3950 2    50   Input ~ 0
 SPI1_MOSI
+Text GLabel 8150 4450 0    50   Input ~ 0
+USART1_TX
 Text GLabel 8650 4450 2    50   Input ~ 0
-USART1_TX
-Text GLabel 8150 4450 0    50   Input ~ 0
 USART1_RX
 NoConn ~ 4550 3750
@@
 Connection ~ 8650 3650
 $Comp
-L power:GND #PWR?
+L power:GND #PWR0101
 U 1 1 610634B2
 P 8900 4050
-F 0 "#PWR?" H 8900 3800 50  0001 C CNN
+F 0 "#PWR0101" H 8900 3800 50  0001 C CNN
 F 1 "GND" V 8905 3922 50  0000 R CNN
 F 2 "" H 8900 4050 50  0001 C CNN
@@
 $EndComp
 $Comp
-L power:GND #PWR?
+L power:GND #PWR0102
 U 1 1 6106372B
 P 7850 4050
-F 0 "#PWR?" H 7850 3800 50  0001 C CNN
+F 0 "#PWR0102" H 7850 3800 50  0001 C CNN
 F 1 "GND" V 7855 3922 50  0000 R CNN
 F 2 "" H 7850 4050 50  0001 C CNN
@@
 	8650 4050 8900 4050
 $Comp
-L power:+3.3V #PWR?
+L power:+3.3V #PWR0103
 U 1 1 61065C5C
 P 7550 4350
-F 0 "#PWR?" H 7550 4200 50  0001 C CNN
+F 0 "#PWR0103" H 7550 4200 50  0001 C CNN
 F 1 "+3.3V" H 7565 4523 50  0000 C CNN
 F 2 "" H 7550 4350 50  0001 C CNN
@@
 	7550 4350 8150 4350
 $Comp
-L power:GND #PWR?
+L power:GND #PWR0104
 U 1 1 6106A77D
 P 8900 4350
-F 0 "#PWR?" H 8900 4100 50  0001 C CNN
+F 0 "#PWR0104" H 8900 4100 50  0001 C CNN
 F 1 "GND" V 8905 4222 50  0000 R CNN
 F 2 "" H 8900 4350 50  0001 C CNN
@@
 Wire Wire Line
 	8650 4350 8900 4350
+Wire Wire Line
+	5600 3950 6200 3950
+Wire Wire Line
+	5600 3850 6100 3850
+Wire Wire Line
+	6100 3800 6100 3850
+Connection ~ 6100 3850
+Wire Wire Line
+	6100 3850 6550 3850
+Wire Wire Line
+	6200 3800 6200 3950
+Connection ~ 6200 3950
+Wire Wire Line
+	6200 3950 6550 3950
 $EndSCHEMATC
